File: schematics/smart_clock.sch (KiCad schematic (older format))
At the start: 6 parts

Commit message: Schematics added.
Parts:
- added U1: DT-06_WiFi_Board, symbol mrach_custom:DT-06_WiFi_Board
- gave numbers to parts that had none: 6
Connections:
- net GND: now also U2.10 (GND), U2.11 (GND), U2.12 (GND), U2.13 (GND), U2.5 (GND), U2.6 (GND), U2.7 (GND), U2.8 (GND), U2.9 (GND), U3.4 (GND), U1.~ (VCC)
- net at A1.5V1 (5V): now also U2.2 (VCC), U3.1 (VCC), U1.~ (VCC)
- net at A1.D18 (D18_TX1): now also U1.~ (VCC)
- net at A1.D19 (D19_RX1): now also U1.~ (VCC)
Other:
- note added: "Real Time Clock module"
- note added: "TFT Screen 320x480 HX8357B Arduino MEGA Shield"
- note added: "Temperature sensor"
- note added: "WiFi module"
- moved on the sheet: J1, U2, U3

Commit message: Ambient light sensor added. Hours/minutes adjustment buttons added.
Additionally - fixed potential issue with the RTC timer freezing on
battery power.
Parts:
- removed SW1: Dimming Switch, symbol Switch:SW_SPST
- added R2: R150-300k, symbol Device:R_PHOTO
- added SW1, SW2: SW_DPST_x2, symbol Switch:SW_DPST_x2
- A1: symbol mrach_custom:Arduino_Mega2560 -> smart_clock-rescue:Arduino_Mega2560-mrach_custom-smart_clock-rescue
- R1: value 10k -> R270k
- U1: symbol mrach_custom:DT-06_WiFi_Board -> smart_clock-rescue:DT-06_WiFi_Board-mrach_custom-smart_clock-rescue
Connections:
- net GND: no longer R1.2
- net at A1.5V1 (5V), U1.~ (VCC), U2.2 (VCC)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: now also R1.2
- net at A1.A0: now also R1.1, R2.1
- net at A1.D10: now also SW1.1 (A)
- net at A1.D11: now also SW1.3 (A)
- net at A1.D12: now also SW2.1 (A)
- net at A1.D13: now also SW2.3 (A)
- net at A1.D7: no longer R1.1
- net at A1.GND1 (GND): now also R2.2
- net at A1.GND4 (SPI_GND): now also SW1.2 (B), SW1.4 (B), SW2.2 (B), SW2.4 (B)
Other:
- note added: "Joystick buttons"
- note added: "Light sensor"
- moved on the sheet: U2, U3
Changed lines of the file:
@@
 $EndDescr
 $Comp
-L mrach_custom:Arduino_Mega2560 A1
+L smart_clock-rescue:Arduino_Mega2560-mrach_custom-smart_clock-rescue A1
 U 1 1 5CAA5EC6
 P 4700 3400
@@
 Text Notes 1400 6050 0    50   ~ 0
 Power is received from the built-in \nUSB socket of Arduino Mega
-Wire Wire Line
-	6000 1750 7750 1750
-$Comp
-L Device:R R1
-U 1 1 5CAEB1EE
-P 7750 2400
-F 0 "R1" H 7820 2446 50  0000 L CNN
-F 1 "10k" H 7820 2355 50  0000 L CNN
-F 2 "" V 7680 2400 50  0001 C CNN
-F 3 "~" H 7750 2400 50  0001 C CNN
-	1    7750 2400
-	1    0    0    -1
-$EndComp
-Wire Wire Line
-	7750 2550 7750 2750
-$Comp
-L power:GND #PWR04
-U 1 1 5CAEBC68
-P 7750 2750
-F 0 "#PWR04" H 7750 2500 50  0001 C CNN
-F 1 "GND" H 7755 2577 50  0000 C CNN
-F 2 "" H 7750 2750 50  0001 C CNN
-F 3 "" H 7750 2750 50  0001 C CNN
-	1    7750 2750
-	1    0    0    -1
-$EndComp
-Wire Wire Line
-	7750 2250 7750 1750
-$Comp
-L power:+5V #PWR03
-U 1 1 5CAECAB0
-P 7750 950
-F 0 "#PWR03" H 7750 800 50  0001 C CNN
-F 1 "+5V" H 7765 1123 50  0000 C CNN
-F 2 "" H 7750 950 50  0001 C CNN
-F 3 "" H 7750 950 50  0001 C CNN
-	1    7750 950
-	1    0    0    -1
-$EndComp
-$Comp
-L Switch:SW_SPST SW1
-U 1 1 5CAEEEA5
-P 7750 1450
-F 0 "SW1" V 7796 1362 50  0000 R CNN
-F 1 "Dimming Switch" V 7705 1362 50  0000 R CNN
-F 2 "" H 7750 1450 50  0001 C CNN
-F 3 "~" H 7750 1450 50  0001 C CNN
-	1    7750 1450
-	0    -1   -1   0
-$EndComp
-Wire Wire Line
-	7750 1650 7750 1750
-Connection ~ 7750 1750
-Wire Wire Line
-	7750 1250 7750 950
 $Comp
 L Timer_RTC:DS3231M U2
 U 1 1 5CAF1E87
-P 1750 3350
-F 0 "U2" H 1750 2861 50  0000 C CNN
-F 1 "DS3231M" H 1750 2770 50  0000 C CNN
-F 2 "Package_SO:SOIC-16W_7.5x10.3mm_P1.27mm" H 1750 2750 50  0001 C CNN
-F 3 "http://datasheets.maximintegrated.com/en/ds/DS3231.pdf" H 2020 3400 50  0001 C CNN
-	1    1750 3350
+P 1750 2950
+F 0 "U2" H 1750 2461 50  0000 C CNN
+F 1 "DS3231M" H 1750 2370 50  0000 C CNN
+F 2 "Package_SO:SOIC-16W_7.5x10.3mm_P1.27mm" H 1750 2350 50  0001 C CNN
+F 3 "http://datasheets.maximintegrated.com/en/ds/DS3231.pdf" H 2020 3000 50  0001 C CNN
+	1    1750 2950
 	-1   0    0    -1
 $EndComp
@@
 	7450 5300 10800 5300
 Entry Wire Line
-	6550 2450 6650 2550
-Entry Wire Line
 	6550 2550 6650 2650
 Entry Wire Line
@@
 	3250 4900 1000 4900
 Wire Wire Line
-	1000 4900 1000 2850
+	1000 4900 1000 4650
 Wire Wire Line
 	1000 1450 1800 1450
 Wire Wire Line
-	1800 1450 1800 1700
-Wire Wire Line
-	850  3750 850  2350
+	850  3350 850  2350
 Wire Wire Line
 	850  2350 1800 2350
 Wire Wire Line
-	1800 2350 1800 2300
-Wire Wire Line
-	1000 2850 1850 2850
-Wire Wire Line
-	1850 2850 1850 2950
-Connection ~ 1000 2850
-Wire Wire Line
-	1000 2850 1000 1450
-Wire Wire Line
-	1750 3750 850  3750
+	1000 2500 1850 2500
+Wire Wire Line
+	1850 2500 1850 2550
+Connection ~ 1000 2500
+Wire Wire Line
+	1000 2500 1000 1450
+Wire Wire Line
+	1750 3350 850  3350
 Wire Bus Line
 	6650 5900 8050 5900
@@
 	8050 5900 8050 5300
 $Comp
-L mrach_custom:DT-06_WiFi_Board U1
+L smart_clock-rescue:DT-06_WiFi_Board-mrach_custom-smart_clock-rescue U1
 U 1 1 5CB8F77B
 P 1600 400
@@
 	2950 1650 3400 1650
 Wire Wire Line
-	2950 2000 2950 1650
-Wire Wire Line
-	2100 2000 2950 2000
+	2950 1900 2950 1650
 Wire Wire Line
 	2450 1350 2450 1550
@@
 	6300 5750 6300 6300
 Wire Wire Line
-	2250 3150 2850 3150
-Wire Wire Line
-	2850 3150 2850 2350
+	2250 2750 2850 2750
+Wire Wire Line
+	2850 2750 2850 2350
 Wire Wire Line
 	2850 2350 3400 2350
@@
 	3400 2250 2950 2250
 Wire Wire Line
-	2950 2250 2950 3250
-Wire Wire Line
-	2950 3250 2250 3250
+	2950 2250 2950 2850
+Wire Wire Line
+	2950 2850 2250 2850
 Wire Wire Line
 	2750 5050 2750 5100
@@
 	2750 5050 3400 5050
 Wire Wire Line
-	850  3750 850  5050
-Connection ~ 850  3750
+	850  3350 850  5050
+Connection ~ 850  3350
 Connection ~ 850  5050
 Wire Wire Line
@@
 	850  2350 850  1550
 Wire Wire Line
-	850  1550 2250 1550
-Wire Wire Line
 	2250 1550 2250 1350
 Connection ~ 850  2350
@@
 	2150 1350 2150 1450
 Connection ~ 1800 1450
-Wire Bus Line
-	6650 2550 6650 5900
-$Comp
-L Sensor:DHT11 U3
-U 1 1 5CAF1154
-P 1800 2000
-F 0 "U3" H 1556 2046 50  0000 R CNN
-F 1 "DHT22" H 1556 1955 50  0000 R CNN
-F 2 "Sensor:Aosong_DHT11_5.5x12.0_P2.54mm" H 1800 1600 50  0001 C CNN
-F 3 "" H 1950 2250 50  0001 C CNN
-	1    1800 2000
-	1    0    0    -1
-$EndComp
-Text Notes 1900 2350 0    50   ~ 0
+Text Notes 1850 2200 0    50   ~ 0
 Temperature sensor
 Text Notes 1500 1000 0    50   ~ 0
 WiFi module
-Text Notes 2000 3800 0    50   ~ 0
+Text Notes 1850 3400 0    50   ~ 0
 Real Time Clock module
+$Comp
+L Switch:SW_DPST_x2 SW2
+U 2 1 5D6E8061
+P 7350 2350
+F 0 "SW2" H 7350 2585 50  0000 C CNN
+F 1 "SW_DPST_x2" H 7350 2494 50  0000 C CNN
+F 2 "" H 7350 2350 50  0001 C CNN
+F 3 "~" H 7350 2350 50  0001 C CNN
+	2    7350 2350
+	1    0    0    -1
+$EndComp
+$Comp
+L Switch:SW_DPST_x2 SW2
+U 1 1 5D6E7C0F
+P 7350 2000
+F 0 "SW2" H 7350 2235 50  0000 C CNN
+F 1 "SW_DPST_x2" H 7350 2144 50  0000 C CNN
+F 2 "" H 7350 2000 50  0001 C CNN
+F 3 "~" H 7350 2000 50  0001 C CNN
+	1    7350 2000
+	1    0    0    -1
+$EndComp
+$Comp
+L Switch:SW_DPST_x2 SW1
+U 2 1 5D6E7985
+P 7350 1650
+F 0 "SW1" H 7350 1885 50  0000 C CNN
+F 1 "SW_DPST_x2" H 7350 1794 50  0000 C CNN
+F 2 "" H 7350 1650 50  0001 C CNN
+F 3 "~" H 7350 1650 50  0001 C CNN
+	2    7350 1650
+	1    0    0    -1
+$EndComp
+$Comp
+L Switch:SW_DPST_x2 SW1
+U 1 1 5D6E4E45
+P 7350 1300
+F 0 "SW1" H 7350 1535 50  0000 C CNN
+F 1 "SW_DPST_x2" H 7350 1444 50  0000 C CNN
+F 2 "" H 7350 1300 50  0001 C CNN
+F 3 "~" H 7350 1300 50  0001 C CNN
+	1    7350 1300
+	1    0    0    -1
+$EndComp
+Entry Wire Line
+	6550 2450 6650 2550
+Wire Wire Line
+	6900 1650 7150 1650
+Wire Wire Line
+	7000 2000 7150 2000
+Wire Wire Line
+	4850 800  4850 750
+Wire Wire Line
+	4850 750  7700 750
+Wire Wire Line
+	7700 750  7700 1300
+Wire Wire Line
+	7700 2350 7550 2350
+Wire Wire Line
+	7550 1300 7700 1300
+Connection ~ 7700 1300
+Wire Wire Line
+	7700 1300 7700 1650
+Wire Wire Line
+	7550 1650 7700 1650
+Connection ~ 7700 1650
+Wire Wire Line
+	7700 1650 7700 2000
+Wire Wire Line
+	7550 2000 7700 2000
+Connection ~ 7700 2000
+Wire Wire Line
+	7700 2000 7700 2350
+Wire Wire Line
+	850  1550 2250 1550
+Wire Wire Line
+	1800 2350 1800 2200
+Wire Wire Line
+	2100 1900 2950 1900
+Wire Wire Line
+	1800 1450 1800 1600
+$Comp
+L Sensor:DHT11 U3
+U 1 1 5CAF1154
+P 1800 1900
+F 0 "U3" H 1556 1946 50  0000 R CNN
+F 1 "DHT22" H 1556 1855 50  0000 R CNN
+F 2 "Sensor:Aosong_DHT11_5.5x12.0_P2.54mm" H 1800 1500 50  0001 C CNN
+F 3 "" H 1950 2150 50  0001 C CNN
+	1    1800 1900
+	1    0    0    -1
+$EndComp
+$Comp
+L Device:R_PHOTO R2
+U 1 1 5D762175
+P 2850 4650
+F 0 "R2" V 3057 4650 50  0000 C CNN
+F 1 "R150-300k" V 2966 4650 50  0000 C CNN
+F 2 "" V 2900 4400 50  0001 L CNN
+F 3 "~" H 2850 4600 50  0001 C CNN
+	1    2850 4650
+	0    -1   -1   0
+$EndComp
+Wire Wire Line
+	3000 4650 3400 4650
+$Comp
+L Device:R R1
+U 1 1 5D7674A4
+P 2000 4650
+F 0 "R1" V 1793 4650 50  0000 C CNN
+F 1 "R270k" V 1884 4650 50  0000 C CNN
+F 2 "" V 1930 4650 50  0001 C CNN
+F 3 "~" H 2000 4650 50  0001 C CNN
+	1    2000 4650
+	0    1    1    0
+$EndComp
+Wire Wire Line
+	2150 4650 2350 4650
+Wire Wire Line
+	2350 4650 2350 4250
+Wire Wire Line
+	2350 4250 3100 4250
+Wire Wire Line
+	3100 4250 3100 2550
+Wire Wire Line
+	3100 2550 3400 2550
+Connection ~ 2350 4650
+Wire Wire Line
+	2350 4650 2700 4650
+Wire Wire Line
+	1850 4650 1000 4650
+Connection ~ 1000 4650
+Wire Wire Line
+	1000 4650 1000 2500
+Text Notes 1300 4550 0    50   ~ 0
+Light sensor
+Text Notes 7050 2550 0    50   ~ 0
+Joystick buttons
+Wire Wire Line
+	6000 2350 7150 2350
+Wire Wire Line
+	7000 2000 7000 2250
+Wire Wire Line
+	7000 2250 6000 2250
+Wire Wire Line
+	6900 1650 6900 2150
+Wire Wire Line
+	6900 2150 6000 2150
+Wire Wire Line
+	6800 1300 6800 2050
+Wire Wire Line
+	6800 2050 6000 2050
+Wire Wire Line
+	6800 1300 7150 1300
+Wire Bus Line
+	6650 2550 6650 5900
 $EndSCHEMATC
